File: alti/alti.kicad_sch (KiCad schematic)
At the start: 11 parts, among them J2 PINHD_1x2_Female, J3 10118193-0001LF, U1 ESP32-S3-WROOM-1-N8R8, U2 TLV75533PDYDR, U3 BMP384, U5 MPU-6500, U6 W25Q128JVSIQ

Commit message: BOM
Parts:
- J2, S1, S2: now left out of the parts list
- J3: DigiKey_Part_Number (none) -> 609-4616-1-ND
- R5, R6: DigiKey_Part_Number (none) -> YAG3394CT-ND
- U1: PACKAGE SMD-41 Espressif Systems -> (none)
- U2, U3: DigiKey_Part_Number (none) -> 296-TLV75533PDYDRCT-ND
- U5: AVAILABILITY (none) -> In Stock; Availability In Stock -> (none); DigiKey_Part_Number (none) -> 1428-1011-1-ND; PRICE (none) -> None; Price None -> (none)
Changed lines of the file:
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@@
+			)
+		)
+		(property "DigiKey_Part_Number" "296-TLV75533PDYDRCT-ND"
+			(at 147.32 95.25 0)
+			(hide yes)
+			(show_name no)
+			(do_not_autoplace no)
+			(effects
+				(font
+					(size 1.27 1.27)
+				)
 			)
 		)
@@
 			)
 		)
+		(property "DigiKey_Part_Number" "296-TLV75533PDYDRCT-ND "
+			(at 207.01 54.61 0)
+			(hide yes)
+			(show_name no)
+			(do_not_autoplace no)
+			(effects
+				(font
+					(size 1.27 1.27)
+				)
+			)
+		)
 		(pin "10"
 		)
@@
 			)
 		)
+		(property "DigiKey_Part_Number" "YAG3394CT-ND"
+			(at 204.47 106.68 0)
+			(hide yes)
+			(show_name no)
+			(do_not_autoplace no)
+			(effects
+				(font
+					(size 1.27 1.27)
+				)
+			)
+		)
 		(pin "1"
 		)
@@
 			)
 		)
-		(property "PACKAGE" "SMD-41 Espressif Systems"
+		(property "Package" "SMD-41 Espressif Systems"
 			(at 60.96 77.47 0)
 			(hide yes)
@@
 			)
 		)
+		(property "DigiKey_Part_Number" "YAG3394CT-ND"
+			(at 204.47 104.14 0)
+			(hide yes)
+			(show_name no)
+			(do_not_autoplace no)
+			(effects
+				(font
+					(size 1.27 1.27)
+				)
+			)
+		)
 		(pin "1"
 		)
@@
 			)
 		)
-		(property "Price" "None"
+		(property "PRICE" "None"
 			(at 78.74 154.94 0)
 			(hide yes)
@@
 			)
 		)
-		(property "Availability" "In Stock"
+		(property "AVAILABILITY" "In Stock"
 			(at 78.74 154.94 0)
 			(hide yes)
@@
 				)
 				(justify bottom)
+			)
+		)
+		(property "DigiKey_Part_Number" "1428-1011-1-ND"
+			(at 78.74 154.94 0)
+			(hide yes)
+			(show_name no)
+			(do_not_autoplace no)
+			(effects
+				(font
+					(size 1.27 1.27)
+				)
 			)
 		)
@@
 		(body_style 1)
 		(exclude_from_sim no)
-		(in_bom yes)
+		(in_bom no)
 		(on_board yes)
 		(in_pos_files yes)
@@
 		(body_style 1)
 		(exclude_from_sim no)
-		(in_bom yes)
+		(in_bom no)
 		(on_board yes)
 		(in_pos_files yes)
@@
 			)
 		)
+		(property "DigiKey_Part_Number" "609-4616-1-ND"
+			(at 199.39 29.21 0)
+			(hide yes)
+			(show_name no)
+			(do_not_autoplace no)
+			(effects
+				(font
+					(size 1.27 1.27)
+				)
+			)
+		)
 		(pin "2"
 		)
@@
 		(body_style 1)
 		(exclude_from_sim no)
-		(in_bom yes)
+		(in_bom no)
 		(on_board yes)
 		(in_pos_files yes)
@@
 			)
 		)
+		(property "Field16" ""
+			(at 120.65 44.45 0)
+			(hide yes)
+			(show_name no)
+			(do_not_autoplace no)
+			(effects
+				(font
+					(size 1.27 1.27)
+				)
+			)
+		)
